File: Hardware/KiCad/Arduino TPS Enclosure/Arduino TPS Enclosure/Arduino TPS Front.kicad_pcb (KiCad board)
At the start: 2 copper layers, 73.7 x 94 mm, 0 parts

Commit message: Update
Other:
- outline, holes or cut-outs redrawn
- board text added: "1"
- board text added: "2"
- board text added: "3"
- board text added: "4"
- board text added: "Analog"
- board text added: "Arduino-TPS"
- board text added: "Aussparung für die Wiederstände"
- board text added: "Die Tasten sind biegbar, somit können die Tasten gedrückt werden. Die Rückseite ist lötbar um eventuelle Messfehler mit Lötkleckse zu korrigieren"
- board text added: "Input"
- board text added: "Output"
- board text added: "PRG"
- board text added: "PWM"
- board text added: "Platine ist so groß wie die Base und hat keine Lötfläche für den Rahmen. Die Front kann man abschrauben"
- board text added: "S1"
- board text added: "S2"
- board text added: "SEL"
- board text added: "Zugriff auf das Batteriefach"
- board text added: "Zugriff auf die Pins vom Arduino"
