File: Hardware/KiCad/Arduino TPS Enclosure/Arduino TPS Enclosure/Arduino TPS Base.kicad_pcb (KiCad board)
At the start: 2 copper layers, 73.7 x 91.4 mm, 3 parts

Commit message: Update
Parts:
- moved REF** 2.54 mm to (91.4, 45.7)
- moved REF** 2.54 mm to (82.1, 50.5)
- moved Vin 2.54 mm to (71.1, 109.2)
- renumbered REF** to Vin
Other:
- board size 73.7 x 91.4 mm -> 73.7 x 94 mm
Changed lines of the file:
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@@
 			(outputformat 1)
 			(mirror no)
-			(drillshape 1)
+			(drillshape 0)
 			(scaleselection 1)
-			(outputdirectory "")
+			(outputdirectory "C:/Users/dragon1/Desktop/Gerber")
 		)
 	)
@@
 	(footprint "Connector_PinHeader_2.54mm:PinHeader_1x02_P2.54mm_Vertical"
 		(layer "F.Cu")
-		(at 71.12 106.68 90)
+		(at 71.12 109.22 90)
 		(descr "Through hole straight pin header, 1x02, 2.54mm pitch, single row")
 		(tags "Through hole pin header THT 1x02 2.54mm single row")
-		(property "Reference" "REF**"
+		(property "Reference" "Vin"
 			(at 0 -2.38 90)
 			(layer "F.SilkS")
@@
 			(at 0 4.92 90)
 			(layer "F.Fab")
+			(hide yes)
 			(effects
 				(font
@@
 	(footprint "Button_Switch_THT:SW_E-Switch_EG1224_SPDT_Angled"
 		(layer "F.Cu")
-		(at 91.44 43.18 90)
+		(at 91.44 45.72 90)
 		(descr "E-Switch slide switch, EG series, SPDT, right angle, http://spec_sheets.e-switch.com/specs/P040042.pdf")
 		(tags "switch SPDT")
@@
 	(footprint "Battery:BatteryHolder_Eagle_12BH611-GR"
 		(layer "F.Cu")
-		(at 82.08 47.93)
+		(at 82.08 50.47)
 		(descr "https://eu.mouser.com/datasheet/2/209/EPD-200766-1274481.pdf")
 		(tags "9V Battery Holder")
@@
 			)
 		)
-		(fp_text user "${REFERENCE}"
+		(fp_text user "Battery"
 			(at -24.13 -6.35 0)
 			(layer "F.Fab")
@@
 		)
 	)
+	(gr_rect
+		(start 25.4 25.4)
+		(end 99.06 27.94)
+		(stroke
+			(width 0.2)
+			(type solid)
+		)
+		(fill yes)
+		(layer "F.Cu")
+	)
+	(gr_rect
+		(start 25.4 25.4)
+		(end 27.94 119.38)
+		(stroke
+			(width 0.2)
+			(type solid)
+		)
+		(fill yes)
+		(layer "F.Cu")
+	)
+	(gr_rect
+		(start 25.4 116.84)
+		(end 99.06 119.38)
+		(stroke
+			(width 0.2)
+			(type solid)
+		)
+		(fill yes)
+		(layer "F.Cu")
+	)
+	(gr_rect
+		(start 96.52 25.4)
+		(end 99.06 119.38)
+		(stroke
+			(width 0.2)
+			(type solid)
+		)
+		(fill yes)
+		(layer "F.Cu")
+	)
+	(gr_poly
+		(pts
+			(xy 25.4 25.4) (xy 27.94 25.4) (xy 27.94 119.38) (xy 25.4 119.38)
+		)
+		(stroke
+			(width 0.1)
+			(type solid)
+		)
+		(fill yes)
+		(layer "F.Mask")
+	)
+	(gr_poly
+		(pts
+			(xy 99.06 25.4) (xy 99.06 27.94) (xy 25.4 27.94) (xy 25.4 25.4)
+		)
+		(stroke
+			(width 0.1)
+			(type solid)
+		)
+		(fill yes)
+		(layer "F.Mask")
+	)
+	(gr_poly
+		(pts
+			(xy 99.06 25.4) (xy 99.06 119.38) (xy 96.52 119.38) (xy 96.52 25.4)
+		)
+		(stroke
+			(width 0.1)
+			(type solid)
+		)
+		(fill yes)
+		(layer "F.Mask")
+	)
+	(gr_poly
+		(pts
+			(xy 99.06 119.38) (xy 25.4 119.38) (xy 25.4 116.84) (xy 99.06 116.84)
+		)
+		(stroke
+			(width 0.1)
+			(type solid)
+		)
+		(fill yes)
+		(layer "F.Mask")
+	)
 	(gr_line
-		(start 93.98 71.12)
-		(end 96.52 73.66)
+		(start 93.98 73.66)
+		(end 96.52 76.2)
 		(stroke
 			(width 0.1)
@@
 	)
 	(gr_line
-		(start 96.52 106.68)
-		(end 96.52 73.66)
+		(start 96.52 109.22)
+		(end 96.52 76.2)
 		(stroke
 			(width 0.1)
@@
 	)
 	(gr_line
-		(start 93.98 58.42)
-		(end 93.98 71.12)
+		(start 93.98 60.96)
+		(end 93.98 73.66)
 		(stroke
 			(width 0.1)
@@
 	)
 	(gr_line
-		(start 27.94 58.42)
-		(end 93.98 58.42)
+		(start 27.94 60.96)
+		(end 93.98 60.96)
 		(stroke
 			(width 0.1)
@@
 	)
 	(gr_line
-		(start 27.94 111.75)
+		(start 27.94 114.29)
+		(end 93.98 114.3)
+		(stroke
+			(width 0.1)
+			(type solid)
+		)
+		(layer "F.SilkS")
+	)
+	(gr_line
+		(start 93.98 114.3)
 		(end 93.98 111.76)
 		(stroke
@@
 	)
 	(gr_line
-		(start 93.98 111.76)
-		(end 93.98 109.22)
+		(start 27.94 60.96)
+		(end 27.94 114.29)
 		(stroke
 			(width 0.1)
@@
 	)
 	(gr_line
-		(start 27.94 58.42)
-		(end 27.94 111.75)
-		(stroke
-			(width 0.1)
-			(type solid)
-		)
-		(layer "F.SilkS")
-	)
-	(gr_line
-		(start 96.52 106.68)
-		(end 93.98 109.22)
+		(start 96.52 109.22)
+		(end 93.98 111.76)
 		(stroke
 			(width 0.1)
@@
 	)
 	(gr_line
-		(start 27.94 109.22)
-		(end 22.86 109.22)
+		(start 27.94 111.76)
+		(end 22.86 111.76)
 		(stroke
 			(width 0.05)
@@
 	)
 	(gr_line
-		(start 22.86 109.22)
+		(start 22.86 111.76)
 		(end 22.86 101.6)
 		(stroke
@@
 	(gr_rect
 		(start 25.4 25.4)
-		(end 99.06 116.84)
+		(end 99.06 119.38)
 		(stroke
 			(width 0.05)
@@
 	)
 	(gr_circle
-		(center 27.94 114.3)
-		(end 29.54 114.3)
+		(center 27.94 116.84)
+		(end 29.54 116.84)
 		(stroke
 			(width 0.05)
@@
 	)
 	(gr_circle
-		(center 93.98 104.14)
-		(end 95.58 104.14)
+		(center 93.98 106.68)
+		(end 95.58 106.68)
 		(stroke
 			(width 0.05)
@@
 	)
 	(gr_circle
-		(center 93.98 76.2)
-		(end 95.58 76.2)
+		(center 93.98 78.74)
+		(end 95.58 78.74)
 		(stroke
 			(width 0.05)
@@
 	)
 	(gr_circle
-		(center 43.18 60.96)
-		(end 44.78 60.96)
+		(center 43.18 63.5)
+		(end 44.78 63.5)
 		(stroke
 			(width 0.05)
@@
 	)
 	(gr_circle
-		(center 41.91 109.22)
-		(end 43.51 109.22)
+		(center 41.91 111.76)
+		(end 43.51 111.76)
 		(stroke
 			(width 0.05)
@@
 	)
 	(gr_circle
-		(center 96.52 114.3)
-		(end 98.12 114.3)
+		(center 96.52 116.84)
+		(end 98.12 116.84)
 		(stroke
 			(width 0.05)
@@
 	)
 	(segment
-		(start 82.08 47.93)
-		(end 82.08 90.64)
+		(start 82.08 50.47)
+		(end 82.08 93.18)
 		(width 0.2)
 		(layer "F.Cu")
@@
 	)
 	(segment
-		(start 82.08 90.64)
-		(end 73.66 99.06)
+		(start 82.08 93.18)
+		(end 73.66 101.6)
 		(width 0.2)
 		(layer "F.Cu")
@@
 	)
 	(segment
-		(start 81.28 43.18)
-		(end 78.74 45.72)
+		(start 81.28 45.72)
+		(end 78.74 48.26)
 		(width 0.2)
 		(layer "F.Cu")
@@
 	)
 	(segment
-		(start 82.08 35.23)
-		(end 87.49 35.23)
+		(start 82.08 37.77)
+		(end 87.49 37.77)
 		(width 0.2)
 		(layer "F.Cu")
@@
 	)
 	(segment
-		(start 91.44 43.18)
-		(end 81.28 43.18)
+		(start 91.44 45.72)
+		(end 81.28 45.72)
 		(width 0.2)
 		(layer "F.Cu")
@@
 	)
 	(segment
-		(start 87.49 35.23)
-		(end 91.44 39.18)
+		(start 87.49 37.77)
+		(end 91.44 41.72)
 		(width 0.2)
 		(layer "F.Cu")
@@
 	)
 	(segment
-		(start 78.74 45.72)
-		(end 78.74 88.9)
+		(start 78.74 48.26)
+		(end 78.74 91.44)
 		(width 0.2)
 		(layer "F.Cu")
@@
 	)
 	(segment
-		(start 71.12 96.52)
-		(end 71.12 106.68)
+		(start 71.12 99.06)
+		(end 71.12 109.22)
 		(width 0.2)
 		(layer "F.Cu")
@@
 	)
 	(segment
-		(start 78.74 88.9)
-		(end 71.12 96.52)
+		(start 78.74 91.44)
+		(end 71.12 99.06)
 		(width 0.2)
 		(layer "F.Cu")
@@
 	)
 	(segment
-		(start 73.66 99.06)
-		(end 73.66 106.68)
+		(start 73.66 101.6)
+		(end 73.66 109.22)
 		(width 0.2)
 		(layer "F.Cu")

Commit message: Update
Parts:
- moved REF** 59.5 mm to (32.2, 40.1), turned to -90 degrees
- moved REF** 42.3 mm to (41.9, 37.2), turned to 180 degrees
Routing:
- net (no net): track 151.1 -> 220.1 mm
Other:
- board text added: "+"
- board text added: "-"

Commit message: Update
Parts:
- moved REF** 1.19 mm to (31.0, 40.1)
Routing:
- net (no net): track 220.1 -> 222.5 mm
Other:
- board text added: "GND"
- board text added: "Vin"
- board text removed: "+"
- board text removed: "-"
Changed lines of the file:
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@@
 			(layer "F.Fab")
-		)
-		(fp_text user "${REFERENCE}"
-			(at -2.54 1.27 0)
-			(layer "F.Fab")
-			(effects
-				(font
-					(size 1 1)
-					(thickness 0.15)
-				)
-			)
 		)
 		(pad "1" thru_hole rect
@@
 	(footprint "Button_Switch_THT:SW_E-Switch_EG1224_SPDT_Angled"
 		(layer "F.Cu")
-		(at 32.19 40.1 -90)
+		(at 31 40.1 -90)
 		(descr "E-Switch slide switch, EG series, SPDT, right angle, http://spec_sheets.e-switch.com/specs/P040042.pdf")
 		(tags "switch SPDT")
@@
 		(layer "Edge.Cuts")
 	)
-	(gr_text "+"
-		(at 66.04 109.22 0)
+	(gr_text "Vin"
+		(at 76.2 109.22 0)
 		(layer "F.Cu")
 		(effects
@@
 		)
 	)
-	(gr_text "-"
-		(at 76.2 109.22 0)
+	(gr_text "GND"
+		(at 63.5 109.22 0)
 		(layer "F.Cu")
 		(effects
@@
 	)
 	(segment
-		(start 32.19 44.1)
-		(end 38.04 49.95)
+		(start 31 44.1)
+		(end 32.19 44.1)
+		(width 0.2)
+		(layer "F.Cu")
+		(net 0)
+	)
+	(segment
+		(start 38.04 49.95)
+		(end 41.85 49.95)
 		(width 0.2)
 		(layer "F.Cu")
@@
 	(segment
 		(start 68.04 40.1)
-		(end 32.19 40.1)
+		(end 31 40.1)
 		(width 0.2)
 		(layer "F.Cu")
@@
 	)
 	(segment
-		(start 38.04 49.95)
-		(end 41.85 49.95)
+		(start 32.19 44.1)
+		(end 38.04 49.95)
 		(width 0.2)
 		(layer "F.Cu")
