File: Hardware/KiCad/Arduino TPS/Arduino TPS Front.kicad_pcb (KiCad board)
At the start: 2 copper layers, 73.7 x 94 mm, 0 parts

Commit message: Update
Other:
- board text added: "A0 → Analog 1 A1 → Analog 2 D0 → Input 1 D1 → Input 2 D2 → Input 3 D3 → Input 4 D4 → Output 1 D5 → Output 2 D6 → Output 3 D7 → Output 4 D8 → S2 (PRG) D9 → PWM 1 D10 → PWM 2 D11 → S1 (SEL)"
Changed lines of the file:
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@@
 	)
 	(paper "A5" portrait)
+	(title_block
+		(title "Arduino-TPS Front")
+		(date "2026-02-01")
+		(rev "1.0.0")
+	)
 	(layers
 		(0 "F.Cu" signal)
@@
 	)
 	(gr_text "Aussparung für\ndie Wiederstände"
-		(at 63.5 71.12 0)
+		(at 68.58 68.58 0)
 		(layer "Cmts.User")
 		(effects
@@
 		(effects
 			(font
+				(size 1 1)
+				(thickness 0.15)
+			)
+			(justify left bottom)
+		)
+	)
+	(gr_text "A0  → Analog 1\nA1  → Analog 2\n\nD0  → Input 1\nD1  → Input 2\nD2  → Input 3\nD3  → Input 4\nD4  → Output 1\nD5  → Output 2\nD6  → Output 3\nD7  → Output 4\nD8  → S2 (PRG)\nD9  → PWM 1\nD10 → PWM 2\nD11 → S1 (SEL)"
+		(at 26.5 55.88 0)
+		(layer "Edge.Cuts")
+		(effects
+			(font
