File: Hardware/KiCad/Arduino TPS/Arduino TPS.kicad_pcb (KiCad board)
At the start: 2 copper layers, 19 parts, among them SW3 SW_Push, SW4 SW_Push, SW5 SW_Push, SW6 SW_Push, SW7 SW_Push, SW8 SW_Push

Commit message: Update
Parts:
- added RV1: R_Potentiometer, Library:3310, F.Cu at (81.3, 61.0)
- added RV2: R_Potentiometer, Library:3310, F.Cu at (81.3, 48.3)
- moved SW2 63.8 mm to (116.8, 63.5)
- moved SW3 63.8 mm to (106.7, 63.5)
- moved SW4 63.8 mm to (96.5, 63.5)
- moved SW1 63.7 mm to (127.0, 63.5)
- moved SW6 63.7 mm to (136.0, 75.6)
- moved A1 63.6 mm to (99.1, 83.8)
- moved R1 63.6 mm to (109.2, 45.7)
- moved R2 63.6 mm to (111.8, 40.6)
- moved R3 63.6 mm to (116.8, 45.7)
- moved R4 63.6 mm to (119.4, 40.6)
- moved R5 63.6 mm to (121.9, 45.7)
- moved R6 63.6 mm to (124.5, 40.6)
- moved SW5 63.6 mm to (74.8, 71.1)
- moved D1 63.6 mm to (124.5, 55.9)
- moved D2 63.6 mm to (119.4, 55.9)
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- renumbered SW3 to SW1, SW4 to SW2, SW5 to SW3, SW6 to SW4, SW7 to SW5, SW8 to SW6
Connections:
- A1 pad 29: GNDD -> unconnected-(A1-GND-Pad29)
- A1 pad 6: GNDD -> unconnected-(A1-GND-Pad6)
- A1 pad 7: GNDD -> unconnected-(A1-GND-Pad7)
- D2 pad 2: unconnected-(D2-A-Pad2) -> Net-(D2-A)
- D3 pad 2: unconnected-(D3-A-Pad2) -> Net-(D3-A)
- R4 pad 1: unconnected-(R4-Pad1) -> A3
- R4 pad 2: unconnected-(R4-Pad2) -> Net-(D3-A)
- R5 pad 1: unconnected-(R5-Pad1) -> Net-(D2-A)
- SW5 pad 1: GNDD -> unconnected-(SW5-Pad1)
- SW6 pad 1: GNDD -> unconnected-(SW6-Pad1)
- SW6 pad 2: GNDD -> S2
Routing:
- net Net-(D3-A): track 0.00 -> 12.7 mm
- net (no net): track 12.7 -> 0.00 mm
- net Net-(D2-A): track 0.00 -> 10.2 mm
- net E2: track 38.1 -> 41.8 mm
- net E4: track 48.3 -> 51.9 mm
- net E3: track 40.6 -> 44.3 mm
- net S2: track 105.0 -> 102.5 mm
- net GNDD: track 135.2 -> 134.1 mm
- net S1: track 69.7 -> 70.3 mm
- net E1: track 28.5 -> 29.1 mm

Commit message: Update
Other:
- board outline added: 68.6 x 53.3 mm
Changed lines of the file:
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@@
 			(outputformat 1)
 			(mirror no)
-			(drillshape 1)
+			(drillshape 0)
 			(scaleselection 1)
-			(outputdirectory "")
+			(outputdirectory "Gerber/")
 		)
 	)
@@
 		(net 14)
 	)
+	(gr_line
+		(start 139.7 81.28)
+		(end 137.16 83.82)
+		(stroke
+			(width 0.05)
+			(type default)
+		)
+		(layer "Edge.Cuts")
+	)
+	(gr_line
+		(start 71.12 83.82)
+		(end 71.12 33.02)
+		(stroke
+			(width 0.05)
+			(type default)
+		)
+		(layer "Edge.Cuts")
+	)
+	(gr_line
+		(start 137.16 83.82)
+		(end 137.16 86.36)
+		(stroke
+			(width 0.05)
+			(type default)
+		)
+		(layer "Edge.Cuts")
+	)
+	(gr_line
+		(start 71.12 33.02)
+		(end 137.16 33.02)
+		(stroke
+			(width 0.05)
+			(type default)
+		)
+		(layer "Edge.Cuts")
+	)
+	(gr_line
+		(start 137.16 45.72)
+		(end 139.7 48.26)
+		(stroke
+			(width 0.05)
+			(type default)
+		)
+		(layer "Edge.Cuts")
+	)
+	(gr_line
+		(start 137.16 33.02)
+		(end 137.16 45.72)
+		(stroke
+			(width 0.05)
+			(type default)
+		)
+		(layer "Edge.Cuts")
+	)
+	(gr_line
+		(start 139.7 48.26)
+		(end 139.7 81.28)
+		(stroke
+			(width 0.05)
+			(type default)
+		)
+		(layer "Edge.Cuts")
+	)
+	(gr_line
+		(start 71.12 86.36)
+		(end 71.12 83.82)
+		(stroke
+			(width 0.05)
+			(type default)
+		)
+		(layer "Edge.Cuts")
+	)
+	(gr_line
+		(start 137.16 86.36)
+		(end 71.12 86.36)
+		(stroke
+			(width 0.05)
+			(type default)
+		)
+		(layer "Edge.Cuts")
+	)
 	(segment

Commit message: Update
Parts:
- RV1: value R_Potentiometer -> AD1
- RV2: value R_Potentiometer -> AD2
Changed lines of the file:
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@@
 		(date "2026-02-01")
 		(rev "2.0.0")
-		(comment 1 "Tastenprogrammierbare Steuerung")
 	)
 	(layers
@@
 			(at 2.54 2.37 90)
 			(layer "F.Fab")
+			(hide yes)
 			(effects
 				(font
@@
 		)
 		(fp_text user "${REFERENCE}"
-			(at 2.54 -2.37 90)
+			(at 2.54 0 0)
 			(layer "F.Fab")
 			(effects
@@
 			(at 2.54 2.37 90)
 			(layer "F.Fab")
+			(hide yes)
 			(effects
 				(font
@@
 		)
 		(fp_text user "${REFERENCE}"
-			(at 2.54 -2.37 90)
+			(at 2.54 0 0)
 			(layer "F.Fab")
 			(effects
@@
 			)
 		)
-		(property "Value" "R_Potentiometer"
-			(at 0 1 0)
+		(property "Value" "AD1"
+			(at 0 0 0)
 			(unlocked yes)
 			(layer "F.Fab")
@@
 			(layer "F.SilkS")
 		)
-		(fp_text user "3310 – 9 mm Square Sealed Panel Control"
-			(at 0 2.5 0)
-			(unlocked yes)
-			(layer "F.Fab")
-			(effects
-				(font
-					(size 1 1)
-					(thickness 0.15)
-				)
-			)
-		)
 		(pad "1" thru_hole circle
 			(at -2.54 2.54)
@@
 			(at 3.75 6.7 0)
 			(layer "F.Fab")
+			(hide yes)
 			(effects
 				(font
@@
 			(layer "F.Fab")
 		)
-		(fp_text user "${REFERENCE}"
+		(fp_text user "S1"
 			(at 3.25 2.25 0)
 			(layer "F.Fab")
@@
 			(at 3.75 6.7 0)
 			(layer "F.Fab")
+			(hide yes)
 			(effects
 				(font
@@
 			(layer "F.Fab")
 		)
-		(fp_text user "${REFERENCE}"
+		(fp_text user "E2"
 			(at 3.25 2.25 0)
 			(layer "F.Fab")
@@
 			(at 2.54 2.37 90)
 			(layer "F.Fab")
+			(hide yes)
 			(effects
 				(font
@@
 		)
 		(fp_text user "${REFERENCE}"
-			(at 2.54 -2.37 90)
+			(at 2.54 0 0)
 			(layer "F.Fab")
 			(effects
@@
 			(at 2.54 2.37 90)
 			(layer "F.Fab")
+			(hide yes)
 			(effects
 				(font
@@
 		)
 		(fp_text user "${REFERENCE}"
-			(at 2.54 -2.37 90)
+			(at 2.54 0 0)
 			(layer "F.Fab")
 			(effects
@@
 			(layer "F.Fab")
 		)
-		(fp_text user "${REFERENCE}"
-			(at 1.27 -2.667 90)
+		(fp_text user "A2"
+			(at 1.27 0 0)
 			(layer "F.Fab")
 			(effects
@@
 			(at 3.75 6.7 0)
 			(layer "F.Fab")
+			(hide yes)
 			(effects
 				(font
@@
 			(layer "F.Fab")
 		)
-		(fp_text user "${REFERENCE}"
+		(fp_text user "E3"
 			(at 3.25 2.25 0)
 			(layer "F.Fab")
@@
 			(layer "F.Fab")
 		)
-		(fp_text user "${REFERENCE}"
-			(at 1.27 -2.667 90)
+		(fp_text user "A4"
+			(at 1.27 0 0)
 			(layer "F.Fab")
 			(effects
@@
 			(layer "F.Fab")
 		)
-		(fp_text user "${REFERENCE}"
-			(at 1.27 -2.667 90)
+		(fp_text user "A1"
+			(at 1.27 0 0)
 			(layer "F.Fab")
 			(effects
@@
 			(at 3.75 6.7 0)
 			(layer "F.Fab")
+			(hide yes)
 			(effects
 				(font
@@
 			(layer "F.Fab")
 		)
-		(fp_text user "${REFERENCE}"
+		(fp_text user "E1"
 			(at 3.25 2.25 0)
 			(layer "F.Fab")
@@
 			(at 3.75 6.7 0)
 			(layer "F.Fab")
+			(hide yes)
 			(effects
 				(font
@@
 			(layer "F.Fab")
 		)
-		(fp_text user "${REFERENCE}"
+		(fp_text user "E4"
 			(at 3.25 2.25 0)
 			(layer "F.Fab")
@@
 			(layer "F.Fab")
 		)
-		(fp_text user "${REFERENCE}"
-			(at 1.27 -2.667 90)
+		(fp_text user "PWM2"
+			(at 1.27 0 0)
 			(layer "F.Fab")
 			(effects
@@
 			(at 2.54 2.37 90)
 			(layer "F.Fab")
+			(hide yes)
 			(effects
 				(font
@@
 		)
 		(fp_text user "${REFERENCE}"
-			(at 2.54 -2.37 90)
+			(at 2.54 0 0)
 			(layer "F.Fab")
 			(effects
@@
 			)
 		)
-		(property "Value" "R_Potentiometer"
-			(at 0 1 0)
+		(property "Value" "AD2"
+			(at 0 0 0)
 			(unlocked yes)
 			(layer "F.Fab")
@@
 			(layer "F.SilkS")
 		)
-		(fp_text user "3310 – 9 mm Square Sealed Panel Control"
-			(at 0 2.5 0)
-			(unlocked yes)
-			(layer "F.Fab")
-			(effects
-				(font
-					(size 1 1)
-					(thickness 0.15)
-				)
-			)
-		)
 		(pad "1" thru_hole circle
 			(at -2.54 2.54)
@@
 			(layer "F.Fab")
 		)
-		(fp_text user "${REFERENCE}"
-			(at 1.27 -2.667 90)
+		(fp_text user "PWM1"
+			(at 1.27 0 0)
 			(layer "F.Fab")
 			(effects
@@
 			(at 2.54 2.37 90)
 			(layer "F.Fab")
+			(hide yes)
 			(effects
 				(font
@@
 		)
 		(fp_text user "${REFERENCE}"
-			(at 2.54 -2.37 90)
+			(at 2.54 0 0)
 			(layer "F.Fab")
 			(effects
@@
 			(at 3.75 6.7 0)
 			(layer "F.Fab")
+			(hide yes)
 			(effects
 				(font
@@
 			(layer "F.Fab")
 		)
-		(fp_text user "${REFERENCE}"
+		(fp_text user "S2"
 			(at 3.25 2.25 0)
 			(layer "F.Fab")
@@
 			(layer "F.Fab")
 		)
-		(fp_text user "${REFERENCE}"
-			(at 1.27 -2.667 90)
+		(fp_text user "A3"
+			(at 1.27 0 0)
 			(layer "F.Fab")
 			(effects
@@
 			(at 0 -22.86 0)
 			(layer "B.Fab")
+			(hide yes)
 			(effects
 				(font
@@
 			(layer "B.Fab")
 		)
-		(fp_text user "${REFERENCE}"
-			(at 0 -20.32 0)
-			(layer "B.Fab")
-			(effects
-				(font
-					(size 1 1)
-					(thickness 0.15)
-				)
-				(justify mirror)
-			)
-		)
 		(pad "1" thru_hole rect

Commit message: Update
Other:
- outline, holes or cut-outs redrawn
- copper layers 2 -> 10
- board text added: "3.3V"
- board text added: "5V"
- board text added: "A0"
- board text added: "A1"
- board text added: "A2"
- board text added: "A3"
- board text added: "A4"
- board text added: "A5"
- board text added: "AREF"
- board text added: "D0"
- board text added: "D1"
- board text added: "D10"
- board text added: "D11"
- board text added: "D12"
- board text added: "D13"
- board text added: "D2"
- board text added: "D3"
- board text added: "D4"
- board text added: "D5"
- board text added: "D6"
- board text added: "D7"
- board text added: "D8"
- board text added: "D9"
- board text added: "GND"
- board text added: "IOREF"
- board text added: "RESET"
- board text added: "SCL"
- board text added: "SDA"
- board text added: "Vin"
