File: Hardware/KiCad/Arduino TPS/Arduino TPS.kicad_sch (KiCad schematic)
At the start: 21 parts, among them SW1 RotaryEncoder, SW2 RotaryEncoder, SW3 SW_Push, SW4 SW_Push, SW5 SW_Push, SW6 SW_Push, SW7 SW_Push, SW8 SW_Push

Commit message: Update
Parts:
- removed SW1, SW2: RotaryEncoder, symbol Device:RotaryEncoder
- added RV1, RV2: R_Potentiometer, Library:3310, symbol Device:R_Potentiometer
- SW1: renamed from SW3; symbol Switch:SW_MEC_5G -> Switch:SW_MEC_5E
- SW2: renamed from SW4; symbol Switch:SW_MEC_5G -> Switch:SW_MEC_5E
- SW3: renamed from SW5; symbol Switch:SW_MEC_5G -> Switch:SW_MEC_5E
- SW4: renamed from SW6; symbol Switch:SW_MEC_5G -> Switch:SW_MEC_5E
- SW5: renamed from SW7; symbol Switch:SW_MEC_5G -> Switch:SW_MEC_5E
- SW6: renamed from SW8; symbol Switch:SW_MEC_5G -> Switch:SW_MEC_5E
Connections:
- net 5V: now also RV1.1, RV2.1
- net A1: now also R6.1; no longer R6.2
- net A2: now also R5.2
- net A3: now also R4.1
- net A4: now also R3.2; no longer R3.1
- net AD1: now also RV1.2
- net AD2: now also RV2.2
- net E1: no longer SW1.4 (B)
- net E2: no longer SW2.4 (B)
- net E3: no longer SW3.4 (B)
- net E4: no longer SW4.4 (B)
- net GNDD: now also SW6.4 (A), RV1.3, RV2.3; no longer A1.29 (GND), A1.6 (GND), A1.7 (GND), SW5.1 (A), SW6.1 (A), SW6.2 (A)
- net PWM1: now also R2.1; no longer R2.2
- net S1: no longer SW5.3 (B)
- net S2: now also SW6.2; no longer SW6.3 (B), SW6.4 (B)
- net at D4.2 (A): now also R3.1; no longer R3.2
- net at D1.2 (A): now also R6.2; no longer R6.1
- net at R4.2: now also D3.2 (A)
- net at D2.2 (A): now also R5.1
- net at D5.2 (A): now also R2.2; no longer R2.1
Other:
- moved on the sheet: D1, D2, D3, D4, D5, D6, R1, R2, R3, R5, R6

Commit message: Update
Other:
- moved on the sheet: A1, D1, D2, D3, D4, D5, D6, R1, R2, R3, R4, R5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
